File: voltage_doubler.kicad_sch (KiCad schematic)
At the start: 10 parts, among them IC1 LT1054CP, J1 Vin = 3.5V to 15V, J2 Barrel_Jack

Commit message: update checklist, add graphics, add date variable
Other:
- title: (none) -> Voltage doubler
Changed lines of the file:
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@@
 	(generator_version "8.0")
 	(paper "A4")
+	(title_block
+		(title "Voltage doubler")
+		(date "${MANUFACTURING_DATE}")
+		(rev "1.0.0")
+	)
 	(junction
 		(at 92.71 95.25)
@@
 	)
 	(junction
+		(at 73.66 83.82)
+		(diameter 0)
+		(color 0 0 0 0)
+	)
+	(junction
 		(at 162.56 77.47)
 		(diameter 0)
@@
 	(wire
 		(pts
+			(xy 69.85 83.82) (xy 73.66 83.82)
+		)
+		(stroke
+			(width 0)
+			(type default)
+		)
+	)
+	(wire
+		(pts
 			(xy 92.71 77.47) (xy 92.71 87.63)
 		)
@@
 	(wire
 		(pts
+			(xy 69.85 85.09) (xy 69.85 83.82)
+		)
+		(stroke
+			(width 0)
+			(type default)
+		)
+	)
+	(wire
+		(pts
 			(xy 92.71 77.47) (xy 114.3 77.47)
 		)
@@
 	(wire
 		(pts
-			(xy 73.66 80.01) (xy 73.66 85.09)
+			(xy 73.66 80.01) (xy 73.66 83.82)
+		)
+		(stroke
+			(width 0)
+			(type default)
+		)
+	)
+	(wire
+		(pts
+			(xy 73.66 83.82) (xy 73.66 85.09)
 		)
 		(stroke
@@
 					(unit 1)
 				)
+			)
+		)
+	)
+	(symbol
+		(lib_id "power:PWR_FLAG")
+		(at 69.85 85.09 180)
+		(unit 1)
+		(exclude_from_sim no)
+		(in_bom yes)
+		(on_board yes)
+		(dnp no)
+		(fields_autoplaced yes)
+		(property "Reference" "#FLG02"
+			(at 69.85 86.995 0)
+			(effects
+				(font
+					(size 1.27 1.27)
+				)
+				(hide yes)
+			)
+		)
+		(property "Value" "PWR_FLAG"
+			(at 69.85 90.17 0)
+			(effects
+				(font
+					(size 1.27 1.27)
+				)
+			)
+		)
+		(property "Footprint" ""
+			(at 69.85 85.09 0)
+			(effects
+				(font
+					(size 1.27 1.27)
+				)
+				(hide yes)
+			)
+		)
+		(property "Datasheet" "~"
+			(at 69.85 85.09 0)
+			(effects
+				(font
+					(size 1.27 1.27)
+				)
+				(hide yes)
+			)
+		)
+		(property "Description" "Special symbol for telling ERC where power comes from"
+			(at 69.85 85.09 0)
+			(effects
+				(font
+					(size 1.27 1.27)
+				)
+				(hide yes)
+			)
+		)
+		(pin "1"
+		)
+		(instances
+			(project "voltage_doubler"
+				(path "/463eb72c-905e-465d-a172-cee5677dd50c"
+					(reference "#FLG02")
+					(unit 1)
+				)
